File: pcb/draft_1-1/pcb/pcb.sch (KiCad schematic (older format))
At the start: 1 part, among them U1 ATSAML21G18B-AUT

Commit message: paper cut out trade study
Parts:
- removed U1: ATSAML21G18B-AUT, Package_QFP:TQFP-48_7x7mm_P0.5mm, symbol MCU_Microchip_SAML:ATSAML21G18B-AUT
- added BT1: Battery, lir2032:LIR2032, symbol Device:Battery
- added C1: 4.5nF, symbol Device:C
- added C2, C3, C4, C5: C, symbol Device:C
- added FB1: Ferrite_Bead_Small, symbol Device:Ferrite_Bead_Small
- added FID1, FID2, FID3: Fiducial, Fiducial:Fiducial_0.5mm_Mask1mm, symbol Mechanical:Fiducial
- added IC1: BQ21061YFPR, BQ25155:BGA20C40P4X5_162X202X50, symbol BQ25155:BQ21061YFPR
- added J1: XF2M-2415-1A, XF2M-2415-1A:OMRON_XF2M-2415-1A, symbol XF2M-2415-1A:XF2M-2415-1A
- added J2: 10118194-0001LF, 10118194-0001LF:AMPHENOL_10118194-0001LF, symbol 10118194-0001LF:10118194-0001LF
- added LS2: SP-1511S-6, SP-1511S-6:SP-1511S-6_ALT, symbol SP-1511S-6:SP-1511S-6
- added R3: 1M, symbol Device:R
- added S1: TL3315NF100Q, TL3315NF100Q:TL3315NF100Q, symbol TL3315NF100Q:TL3315NF100Q
- added TP1: VREF, symbol Connector:TestPoint
- added TP2: SWDIO, symbol Connector:TestPoint
- added TP3: SWCLK, symbol Connector:TestPoint
- added TP4: ~RESET, symbol Connector:TestPoint
- added TP5: GND, symbol Connector:TestPoint
- added U1: ATSAML21J18B-AUT, Package_QFP:TQFP-64_10x10mm_P0.5mm, symbol MCU_Microchip_SAML:ATSAML21J18B-AUT
- added U2: TPD4S012DRYR, TPD4S012DRYR:SON50P100X145X60-6N, symbol TPD4S012DRYR:TPD4S012DRYR
- added U3: IIS2DLPC, Package_LGA:LGA-12_2x2mm_P0.5mm, symbol custom:IIS2DLPC
- added U4: AT25SF641, Package_SO:SOIC-8_5.275x5.275mm_P1.27mm, symbol Memory_Flash:AT25SF081-SSHD-X
- added U5: XZMDKCBDDG45S-9, XZMDKCBDDG45S-9:PLCC-4, symbol XZMDKCBDDG45S-9:XZMDKCBDDG45S-9
- added U6: eInk_waveshare_1.54A, custom:eInk_waveshare_1.54A, symbol custom:eInk_waveshare_1.54A
- added Y1: 32K, symbol Device:Crystal
Connections:
- net labels added: +1V8, +3V3, +5V, D+, D-, GND, SCL, SDA, SWCLK, SWDIO, VREF, ~RESET
- wire segments 0 -> 31
Other:
- note added: "A ferrite bead can be added between the main power supply (VDD)\nand VDDANA to prevent digital noise from entering the analog\npower domain. The bead should provide enough impedance\n(e.g. 50Ω at 20MHz and 220Ω at 100MHz) to separate the digital\nand analog power domains. Make sure to select a ferrite\nbead designed for filtering applications with a low DC resistance\nto avoid a large voltage dro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"
- note added: "Accelerometer"
- note added: "LED"
- note added: "Memory"
- note added: "PMIC/LDO"
- note added: "RESET"
- note added: "SWD"
- note added: "Tie circuit GND to shield or USB GND?"
- note added: "USB Input"
- note added: "battery\nbuzzer\nled\nePaper (1.8V?)\nFlash memory\ncapacitive touch\nPMIC/LDO\naccel\n(magn)\nusb\n(solar)\nreset button\npogo: SWD@1.8V [VDDIO, SWCLK, SWDIO, nRESET,GND]\nfiducials\nexternal crystal (precison boost?)"
- note added: "eInk Display"
- note removed: "buzzer\nled\nePaper (1.8V?)\n64 kB memory\ncapacitive touch\nPMIC/LDO\naccel (magn)\nusb\nsolar\nreset button\npogo: SWD@1.8V [VDDIO, SWCLK, SWDIO, nRESET,GND]\nfiducials"

Commit message: paper cutout study
Parts:
- removed LS2: SP-1511S-6, SP-1511S-6:SP-1511S-6_ALT, symbol SP-1511S-6:SP-1511S-6
- added D1, D2, D3, D4: D, Diode_SMD:D_SOD-123, symbol Device:D
- added L1: L, Inductor_SMD:L_1206_3216Metric, symbol Device:L
- added LS1: CMT-8503-90-SMT-TR, CMT-8503-90-SMT-TR:XDCR_CMT-8503-90-SMT-TR, symbol CMT-8503-90-SMT-TR:CMT-8503-90-SMT-TR
- added Q1: SI1308EDL-T1-GE3, Package_TO_SOT_SMD:SOT-323_SC-70, symbol Transistor_FET:ZXM61N03F
Other:
- note added: "Audio"
Changed lines of the file:
@@
-$EndComp
-$Comp
-L SP-1511S-6:SP-1511S-6 LS2
-U 1 1 5E485031
-P 5050 1500
-F 0 "LS2" H 5155 1546 50  0000 L CNN
-F 1 "SP-1511S-6" H 5155 1455 50  0000 L CNN
-F 2 "SP-1511S-6:SP-1511S-6_ALT" H 5050 1500 50  0001 L BNN
-F 3 "18 x 13 x 2.5 mm 300 to 1150 Hz 92 dB Spring Lead Low Profile Micro Speaker" H 5050 1500 50  0001 L BNN
-F 4 "CUI" H 5050 1500 50  0001 L BNN "Field4"
-F 5 "CMS-18138A-SP" H 5050 1500 50  0001 L BNN "Field5"
-F 6 "Good" H 5050 1500 50  0001 L BNN "Field6"
-F 7 "1.93 USD" H 5050 1500 50  0001 L BNN "Field7"
-F 8 "CUI" H 5050 1500 50  0001 L BNN "Field8"
-	1    5050 1500
-	1    0    0    -1
 $EndComp
 $Comp
@@
 Text Notes 3650 4950 0    50   ~ 0
 RESET
+$Comp
+L Transistor_FET:ZXM61N03F Q1
+U 1 1 5E47D615
+P 3250 1250
+F 0 "Q1" H 3454 1296 50  0000 L CNN
+F 1 "SI1308EDL-T1-GE3" H 3454 1205 50  0000 L CNN
+F 2 "Package_TO_SOT_SMD:SOT-323_SC-70" H 3450 1175 50  0001 L CIN
+F 3 "http://www.diodes.com/assets/Datasheets/ZXM61N03F.pdf" H 3250 1250 50  0001 L CNN
+	1    3250 1250
+	1    0    0    -1
+$EndComp
+$Comp
+L Device:L L1
+U 1 1 5E4829F3
+P 2850 1650
+F 0 "L1" H 2903 1696 50  0000 L CNN
+F 1 "L" H 2903 1605 50  0000 L CNN
+F 2 "Inductor_SMD:L_1206_3216Metric" H 2850 1650 50  0001 C CNN
+F 3 "~" H 2850 1650 50  0001 C CNN
+	1    2850 1650
+	1    0    0    -1
+$EndComp
+$Comp
+L CMT-8503-90-SMT-TR:CMT-8503-90-SMT-TR LS1
+U 1 1 5E48786A
+P 6950 3700
+F 0 "LS1" H 7129 3746 50  0000 L CNN
+F 1 "CMT-8503-90-SMT-TR" H 7129 3655 50  0000 L CNN
+F 2 "CMT-8503-90-SMT-TR:XDCR_CMT-8503-90-SMT-TR" H 6950 3700 50  0001 L BNN
+F 3 "CUI Inc." H 6950 3700 50  0001 L BNN
+F 4 "Manufacturer Recommendations" H 6950 3700 50  0001 L BNN "Field4"
+F 5 "3.00mm" H 6950 3700 50  0001 L BNN "Field5"
+F 6 "1.0" H 6950 3700 50  0001 L BNN "Field6"
+	1    6950 3700
+	1    0    0    -1
+$EndComp
+Text Notes 7200 3500 0    50   ~ 0
+Audio
+$Comp
+L Device:D D1
+U 1 1 5E48FD17
+P 6700 3700
+F 0 "D1" V 6654 3779 50  0000 L CNN
+F 1 "D" V 6745 3779 50  0000 L CNN
+F 2 "Diode_SMD:D_SOD-123" H 6700 3700 50  0001 C CNN
+F 3 "~" H 6700 3700 50  0001 C CNN
+	1    6700 3700
+	0    1    1    0
+$EndComp
+$Comp
+L Device:D D2
+U 1 1 5E499567
+P 3200 1750
+F 0 "D2" V 3154 1829 50  0000 L CNN
+F 1 "D" V 3245 1829 50  0000 L CNN
+F 2 "Diode_SMD:D_SOD-123" H 3200 1750 50  0001 C CNN
+F 3 "~" H 3200 1750 50  0001 C CNN
+	1    3200 1750
+	0    1    1    0
+$EndComp
+$Comp
+L Device:D D3
+U 1 1 5E499BDD
+P 3500 1750
+F 0 "D3" V 3454 1829 50  0000 L CNN
+F 1 "D" V 3545 1829 50  0000 L CNN
+F 2 "Diode_SMD:D_SOD-123" H 3500 1750 50  0001 C CNN
+F 3 "~" H 3500 1750 50  0001 C CNN
+	1    3500 1750
+	0    1    1    0
+$EndComp
+$Comp
+L Device:D D4
+U 1 1 5E49A26C
+P 3750 1750
+F 0 "D4" V 3704 1829 50  0000 L CNN
+F 1 "D" V 3795 1829 50  0000 L CNN
+F 2 "Diode_SMD:D_SOD-123" H 3750 1750 50  0001 C CNN
+F 3 "~" H 3750 1750 50  0001 C CNN
+	1    3750 1750
+	0    1    1    0
+$EndComp
 $EndSCHEMATC

Commit message: trade study on speaker
Parts:
- removed C2, C3, C4, C5: C, symbol Device:C
- removed IC1: BQ21061YFPR, BQ25155:BGA20C40P4X5_162X202X50, symbol BQ25155:BQ21061YFPR
- removed Y1: 32K, symbol Device:Crystal
- added C10, C11, C12, C13, C14, C5, C6, C8, C9: 1uF, Capacitor_SMD:C_0603_1608Metric, symbol Device:C_Small
- added C15, C16: 4.7uF, Capacitor_SMD:C_0603_1608Metric, symbol Device:C
- added C17: 22uF, Capacitor_SMD:C_0603_1608Metric, symbol Device:C_Small
- added C18, C19: 10uF, Capacitor_SMD:C_0603_1608Metric, symbol Device:C_Small
- added C2: 2.2uF, symbol Device:C_Small
- added C20, C?: 100nF, symbol Device:C
- added C7: 100nF, Capacitor_SMD:C_0603_1608Metric, symbol Device:C_Small
- added Q2: SI1308EDL-T1-GE3, Package_TO_SOT_SMD:SOT-323_SC-70, symbol Transistor_FET:ZXM61N03F
- added R1, R5, R7, R8: 10k, Resistor_SMD:R_0603_1608Metric, symbol Device:R
- added R2: 3R0, Resistor_SMD:R_0603_1608Metric, symbol Device:R
- added R4: 68R0, Resistor_SMD:R_0603_1608Metric, symbol Device:R
- added R6: 10k, symbol Device:R
- added R?: R, symbol Device:R
- added S2: TL3315NF100Q, TL3315NF100Q:TL3315NF100Q, symbol TL3315NF100Q:TL3315NF100Q
- added TH1: 10k, symbol Device:Thermistor
- added TP10: 1V8, symbol Connector:TestPoint
- added TP11: BAT, symbol Connector:TestPoint
- added TP6: ~MR, symbol Connector:TestPoint
- added TP7: 5V0, symbol Connector:TestPoint
- added TP8: PMID, symbol Connector:TestPoint
- added TP9: 3V3, symbol Connector:TestPoint
- added U7: BQ25155, BQ21061YFPR:BGA20C40P4X5_162X202X50, symbol BQ25155:BQ25155
- BT1: value Battery -> 45mAh
- D1, D2, D3, D4: value D -> MBR0530
- L1: value L -> 68uH
Connections:
- net SCL is gone; now on net SCL_1V8: U3.1 (SCL/SPC)
- net SDA is gone; now on net SDA_1V8: U3.4 (SDA/SDI)
- net +1V8: now also U3.10 (Vdd_IO), U3.9 (Vdd), C19.2, C20.2, R5.2, R7.1, R8.1, TP10.1, U7.D1 (VDD), U7.E1 (VIO)
- net +3V3: now also D1.1 (K), J1.15 (VDDIO), J1.16 (VCI), L1.2, LS1.P, U4.8 (VCC), U5.2 (3V3), C15.1, C18.2, C7.1, TP9.1, U7.D4 (LSLDO)
- net +5V: now also TP7.1, U7.A1 (IN)
- net GND: now also BT1.2 (-), D4.1 (K), J1.17 (VSS), J1.8 (BS), S1.3 (P$2), S1.4 (P$2), U1.22 (GND), U1.33 (GND), U1.47 (GND), U1.54 (GND), U1.7 (GNDANA), U3.5 (NC), U3.6 (GND), U4.4 (GND), C10.2, C11.2, C12.2, C13.2, C14.2, C15.2, C17.1, C18.1, C19.1, C2.2, C20.1, C5.2, C6.2, C7.2, C8.2, C9.2, C?.2, Q2.2 (S), R1.2, R2.2, R6.1, R6.2, TH1.1, TH1.2, U7.A4 (GND), U7.B4 (TS), U7.C3 (NC), U7.C4 (ADCIN)
- net ~RESET: now also R?.2; no longer U1.52 (~RESET)
- net INT_ACC_2: now reaches U3.11 (INT2)
- net INT_ACC_1: now reaches U3.12 (INT1)
- net fCS: now reaches U4.1 (~CS)
- net eDIN: now reaches U4.2 (SO/IO1)
- net eDIN: now also J1.14 (SDI)
- net fSDI: now reaches U4.5 (SI/IO0)
- net at U5.1 (RED): now also R4.2
- net BLUE: now reaches U5.3 (BLUE)
- net GREEN: now reaches U5.4 (GREEN)
- net eRST: now reaches J1.10 (RST)
- net eDC: now reaches J1.11 (D/C)
- net eCS: now reaches J1.12 (CS)
- net eCLK: now reaches J1.13 (SCLK)
- net at J1.18 (VDD): now also C8.1
- net at J1.19 (VPP): now also C9.1
- net eGDR: now reaches J1.2 (GDR)
- net eGDR: now also Q1.1 (G), R1.1
- net at J1.20 (VSH): now also C10.1
- net ePREVGH: now reaches J1.21 (PREVGH)
- net ePREVGH: now also D2.1 (K), C11.1
- net at J1.22 (VSL): now also C12.1
- net ePREVGL: now reaches J1.23 (PREVGL)
- net ePREVGL: now also D3.2 (A), C13.1
- net at J1.24 (VCOM): now also C14.1
- net eRESE: now reaches J1.3 (RESE)
- net eRESE: now also Q1.2 (S), R2.1
- net at J1.4 (VGL): now also C5.1
- net at J1.5 (VGH): now also C6.1
- net eBUSY: now reaches J1.9 (BUSY)
- net at Q1.3 (D): now also D2.2 (A), L1.1, C16.1
- net at LS1.N: now also D1.2 (A), Q2.3 (D)
- net at BT1.1 (+): now also C2.1, TP11.1, U7.A3 (BAT), U7.B3 (BAT)
- net at D3.1 (K): now also D4.2 (A), C16.2
- net SDA_1V8: now reaches U1.59 (PB30)
- net SDA_1V8: now also R7.2, U7.E2 (SDA)
- net SCL_1V8: now reaches U1.60 (PB31)
- net SCL_1V8: now also R8.2, U7.E3 (SCL)
- net at S1.1 (P$1), S1.2 (P$1): now also TP6.1, U7.C1 (~MR)
- new net: C?.1, R?.1, U1.52 (~RESET)
- new net: C17.2, TP8.1, U7.A2 (PMID), U7.B2 (PMID), U7.E4 (VINLS)
- new net: S2.1 (P$1), S2.2 (P$1)
- new net: S2.3 (P$2), S2.4 (P$2)
- new net AUDIO: Q2.1 (G)
- new net INT_PG: R5.1, U7.B1 (~PG)
- new net RED: R4.1
- no-connect marks 0 -> 8
Other:
- note added: "1.54"\nModel A"
- note added: "1V8 or 3V3"
- note added: "4-wire\n8-bit SPI"
- note added: "9-17 (?) pins for capacitive touch"
- note added: ">330 ohms"
- note added: "Alternate: BQ21061\nRemoves ADC"
- note added: "Magnetometer"
- note added: "Ref Wavshare 1.54" ePaper Schematic, Oct 2018\nRef John Loefler Hackaday Project eInk Adapter 164772"
- note added: "SERCOM5 I2C VIN\nPAD[0] SDA PB30\nPAD[1] SCL PB31"
- note added: "ePaper Display"
- note added: "try daisy-chain SPI in HW"
- note added: "uP RESET"
- note added: "~MR~ RESET"
- note removed: "RESET"
- note removed: "eInk Display"
- moved on the sheet: BT1, D2, D3, D4, J1, L1, Q1, S1, U3, U4, U5, U6

Commit message: trade study on speaker
Parts:
- gave numbers to parts that had none: 2
Changed lines of the file:
@@
 1V8 or 3V3
 $Comp
-L Device:C C?
+L Device:C C3
 U 1 1 5E936869
 P 8350 5900
-F 0 "C?" H 8465 5946 50  0000 L CNN
+F 0 "C3" H 8465 5946 50  0000 L CNN
 F 1 "100nF" H 8465 5855 50  0000 L CNN
 F 2 "" H 8388 5750 50  0001 C CNN
@@
 $EndComp
 $Comp
-L power:GND #PWR?
+L power:GND #PWR0105
 U 1 1 5E937211
 P 8350 6050
-F 0 "#PWR?" H 8350 5800 50  0001 C CNN
+F 0 "#PWR0105" H 8350 5800 50  0001 C CNN
 F 1 "GND" H 8355 5877 50  0000 C CNN
 F 2 "" H 8350 6050 50  0001 C CNN
@@
 $EndComp
 $Comp
-L Device:R R?
+L Device:R R9
 U 1 1 5E94127E
 P 8100 5750
-F 0 "R?" V 7893 5750 50  0000 C CNN
+F 0 "R9" V 7893 5750 50  0000 C CNN
 F 1 "R" V 7984 5750 50  0000 C CNN
 F 2 "" V 8030 5750 50  0001 C CNN

Commit message: adding schematic
Other:
- note added: "Possible alt:\nLIS2DH12TR\nhigher current draw\nhalf price"
Changed lines of the file:
@@
 Text Notes 7850 5650 0    50   ~ 0
 >330 ohms
+Text Notes 5850 2050 0    50   ~ 0
+Possible alt:\nLIS2DH12TR\nhigher current draw\nhalf price
 $EndSCHEMATC
